Commit message: slam mapping, conditioner actuating, other fixes

File: ice_resurfacer_description/urdf/ice_resurfacer.urdf.xacro (robot description, xacro)
@@ -107,14 +107,16 @@
         <box size="${cond_len} ${cond_width} ${cond_height}"/>
       </geometry>
-      <material name="red">
+      <material name="black">
         <color rgba="0.8 0.0 0.0 1.0"/>
       </material>
     </visual>
-    <xacro:box_inertia m="200" w="${cond_len}" h="${cond_height}" d="${cond_width}"/>
+    <xacro:box_inertia m="10" w="${cond_len}" h="${cond_height}" d="${cond_width}"/>
   </link>
   <joint name="conditioner_joint" type="prismatic">
     <parent link="base_link"/>
     <child link="conditioner_link"/>
-    <origin xyz="${-chassis_len/2 - 0.25} 0 ${-(chassis_height/2) + 0.1}" rpy="0 0 0"/>    <axis xyz="0 0 1"/> <limit lower="0.0" upper="0.5" effort="1000" velocity="0.5"/>
+    <origin xyz="${-chassis_len/2 - 0.25} 0 ${-(chassis_height/2) + 0.1}" rpy="0 0 0"/>
+    <axis xyz="0 0 -1"/>
+    <limit lower="0.0" upper="0.5" effort="10000" velocity="0.5"/>
   </joint>
   <link name="imu_link"/>
@@ -189,4 +191,5 @@
     </joint>
     <joint name="conditioner_joint">
+      <command_interface name="effort"/>
       <state_interface name="position"/>
       <state_interface name="velocity"/>
@@ -202,7 +205,7 @@
     <mu2>20.0</mu2>
     <fdir1>1 0 0</fdir1>
-    <kp>10000000.0</kp>
-    <kd>1.0</kd>
-    <minDepth>0.005</minDepth>
+    <kp>100000.0</kp>
+    <kd>500.0</kd>
+    <minDepth>0.01</minDepth>
     <maxVel>0.1</maxVel>
   </gazebo>
@@ -212,7 +215,7 @@
     <mu2>20.0</mu2>
     <fdir1>1 0 0</fdir1>
-    <kp>10000000.0</kp>
-    <kd>1.0</kd>
-    <minDepth>0.005</minDepth>
+    <kp>100000.0</kp>
+    <kd>500.0</kd>
+    <minDepth>0.01</minDepth>
     <maxVel>0.1</maxVel>
   </gazebo>
@@ -221,7 +224,7 @@
     <mu2>20.0</mu2>
     <fdir1>1 0 0</fdir1>
-    <kp>10000000.0</kp>
-    <kd>1.0</kd>
-    <minDepth>0.005</minDepth>
+    <kp>100000.0</kp>
+    <kd>500.0</kd>
+    <minDepth>0.01</minDepth>
     <maxVel>0.1</maxVel>
   </gazebo>
@@ -230,7 +233,7 @@
     <mu2>20.0</mu2>
     <fdir1>1 0 0</fdir1>
-    <kp>10000000.0</kp>
-    <kd>1.0</kd>
-    <minDepth>0.005</minDepth>
+    <kp>100000.0</kp>
+    <kd>500.0</kd>
+    <minDepth>0.01</minDepth>
     <maxVel>0.1</maxVel>
   </gazebo>
@@ -264,12 +267,12 @@
         <scan>
           <horizontal>
-            <samples>360</samples>
+            <samples>90</samples>
             <resolution>1.0</resolution>
-            <min_angle>-1.5708</min_angle>
-            <max_angle>1.5708</max_angle>
+            <min_angle>-1.57079</min_angle>
+            <max_angle>1.57079</max_angle>
           </horizontal>
         </scan>
         <range>
-          <min>0.3</min>
+          <min>2.0</min>
           <max>15.0</max>
           <resolution>0.01</resolution>

Commit message: Experimenting with path planning and Nav2

File: ice_resurfacer_description/urdf/ice_resurfacer.urdf.xacro (robot description, xacro)
@@ -119,4 +119,5 @@
     <axis xyz="0 0 -1"/>
     <limit lower="0.0" upper="0.5" effort="10000" velocity="0.5"/>
+    <dynamics damping="50.0" friction="50.0"/>
   </joint>
   <link name="imu_link"/>
@@ -191,7 +192,11 @@
     </joint>
     <joint name="conditioner_joint">
-      <command_interface name="effort"/>
-      <state_interface name="position"/>
-      <state_interface name="velocity"/>
+      <command_interface name="position"/>
+      <state_interface name="position">
+        <param name="initial_value">0.0</param>
+      </state_interface>
+      <state_interface name="velocity">
+        <param name="initial_value">0.0</param>
+      </state_interface>
     </joint>
   </ros2_control>
@@ -247,4 +252,12 @@
     <plugin filename="libgz_ros2_control-system.so" name="gz_ros2_control::GazeboSimROS2ControlPlugin">
       <parameters>$(find ice_resurfacer_description)/config/controllers.yaml</parameters>
+        <gazebo>
+    <plugin filename="libgz_ros2_control-system.so" name="gz_ros2_control::GazeboSimROS2ControlPlugin">
+      <parameters>$(find ice_resurfacer_description)/config/controllers.yaml</parameters>
+      <ros>
+        <remapping>/ackermann_steering_controller/reference:=/cmd_vel</remapping>
+      </ros>
+    </plugin>
+  </gazebo>
     </plugin>
   </gazebo>
@@ -286,3 +299,10 @@
     </sensor>
   </gazebo>
+  <gazebo>
+    <plugin filename="gz-sim-odometry-publisher-system" name="gz::sim::systems::OdometryPublisher">
+      <odom_frame>odom</odom_frame>
+      <robot_base_frame>base_link</robot_base_frame>
+      <odom_publish_frequency>50</odom_publish_frequency>
+    </plugin>
+  </gazebo>
 </robot>
