Commit message: Enhanced world model, uppdated sweeping trajectory start point

File: ice_resurfacer_description/urdf/ice_resurfacer2.urdf.xacro (robot description, xacro)
@@ -213,5 +213,11 @@
   </ros2_control>
   <gazebo reference="base_link">
-    <material>Gazebo/Blue</material>
+    <visual>
+      <material>
+        <ambient>0.0 0.12 0.35 1.0</ambient>
+        <diffuse>0.0 0.12 0.35 1.0</diffuse>
+        <specular>0.1 0.1 0.1 1.0</specular>
+      </material>
+    </visual>
     <mu1>0.2</mu1> <mu2>0.2</mu2>
     <self_collide>false</self_collide>
