Commit message: transformed base frame to z = 0.0

File: ice_resurfacer_description/urdf/ice_resurfacer4.urdf.xacro (robot description, xacro)
@@ -2,5 +2,8 @@
 <robot name="ice_resurfacer" xmlns:xacro="http://ros.org/wiki/xacro">
   <xacro:property name="chassis_len" value="4.04"/>
-  <xacro:property name="chassis_width" value="1.585"/> <xacro:property name="chassis_height" value="2.0"/>   <xacro:property name="chassis_mass" value="3143.0"/>  <xacro:property name="wheel_radius" value="0.386"/>
+  <xacro:property name="chassis_width" value="1.585"/>
+  <xacro:property name="chassis_height" value="2.0"/>
+  <xacro:property name="chassis_mass" value="3143.0"/>
+  <xacro:property name="wheel_radius" value="0.386"/>
   <xacro:property name="wheel_width" value="0.215"/>
   <xacro:property name="wheel_mass" value="50.0"/>
@@ -9,9 +12,10 @@
   <xacro:property name="cond_width" value="2.13"/>
   <xacro:property name="cond_len" value="0.75"/>
-  <!-- NOTE THAT STL LENGTH IS 0.90 -->
   <xacro:property name="cond_height" value="0.3"/>
   <xacro:property name="ground_clearance" value="0.25"/>
-  <xacro:macro name="box_inertia" params="m w h d">
+  <!-- UPGRADED MACRO: Now accepts x, y, z to shift the center of mass independently -->
+  <xacro:macro name="box_inertia" params="m w h d x y z">
     <inertial>
+      <origin xyz="${x} ${y} ${z}" rpy="0 0 0"/>
       <mass value="${m}"/>
       <inertia ixx="${(m/12) * (h*h + d*d)}" ixy="0.0" ixz="0.0"
@@ -28,9 +32,10 @@
     </inertial>
   </xacro:macro>
+  <!-- base_link is now physically located at Z=0 (Ground Level) -->
   <link name="base_link">
     <visual>
-      <origin xyz="-0.2 0.95 0.575" rpy="3.14159 0 0"/>
-      <geometry>
-        <mesh filename="package://ice_resurfacer_description/meshes/Zamboni_body.stl" scale="0.03 0.020 0.025"/>
+      <origin xyz="-0.5 0.0 0.0" rpy="0 0 0"/>
+      <geometry>
+        <mesh filename="package://ice_resurfacer_description/meshes/perfect_body.stl" scale="1 1 1"/>
       </geometry>
       <material name="blue">
@@ -39,11 +44,29 @@
     </visual>
     <collision>
-      <origin xyz="0 0 0.3" rpy="0 0 0"/>
+      <origin xyz="0 0 1.55" rpy="0 0 0"/>
       <geometry>
         <box size="${chassis_len} ${chassis_width} ${chassis_height - 0.6}"/>
       </geometry>
     </collision>
-    <xacro:box_inertia m="${chassis_mass}" w="${chassis_len}" h="${chassis_height}" d="${chassis_width}"/>
-  </link>
+    <xacro:box_inertia m="${chassis_mass}" w="${chassis_len}" h="${chassis_height}" d="${chassis_width}" x="0" y="0" z="1.25"/>
+  </link>
+   <!-- 2. The Water Tank Dummy Link -->
+  <link name="water_tank_link">
+    <visual>
+      <origin xyz="-0.5 0.0 0.0" rpy="0 0 0"/>
+      <geometry>
+        <mesh filename="package://ice_resurfacer_description/meshes/watertank.stl" scale="1 1 1"/>
+      </geometry>
+      <material name="white">
+        <color rgba="0.9 0.9 0.9 1.0"/>
+      </material>
+    </visual>
+  </link>
+  <!-- 3. The Glue (Fixed Joint) -->
+  <joint name="water_tank_joint" type="fixed">
+    <parent link="base_link"/>
+    <child link="water_tank_link"/>
+    <origin xyz="0 0 0" rpy="0 0 0"/>
+  </joint>
   <xacro:macro name="rear_wheel" params="prefix reflect">
     <link name="${prefix}_wheel">
@@ -66,5 +89,6 @@
       <parent link="base_link"/>
       <child link="${prefix}_wheel"/>
-      <origin xyz="${-wheel_base_x} ${reflect * wheel_sep_y} ${wheel_radius - (ground_clearance + chassis_height/2)}" rpy="${-pi/2} 0 0"/>
+      <!-- Appended + 1.25 to the mathematical Z calculation -->
+      <origin xyz="${-wheel_base_x} ${reflect * wheel_sep_y} ${wheel_radius - (ground_clearance + chassis_height/2) + 1.25}" rpy="${-pi/2} 0 0"/>
       <axis xyz="0 0 1"/>
     </joint>
@@ -82,5 +106,6 @@
       <parent link="base_link"/>
       <child link="${prefix}_steering_link"/>
-      <origin xyz="${wheel_base_x} ${reflect * wheel_sep_y} ${wheel_radius - (ground_clearance + chassis_height/2)}" rpy="0 0 0"/>
+      <!-- Appended + 1.25 to the mathematical Z calculation -->
+      <origin xyz="${wheel_base_x} ${reflect * wheel_sep_y} ${wheel_radius - (ground_clearance + chassis_height/2) + 1.25}" rpy="0 0 0"/>
       <axis xyz="0 0 1"/>
       <limit lower="-0.6" upper="0.6" effort="50000" velocity="1.0"/>
@@ -111,5 +136,5 @@
   <link name="conditioner_link">
     <visual>
-      <origin xyz="-0.25 0.0 -0.15" rpy="0 0 1.5708"/>
+      <origin xyz="-0.33 0.0 -0.15" rpy="0 0 1.5708"/>
       <geometry>
         <mesh filename="package://ice_resurfacer_description/meshes/Conditioner.stl" scale="1.0 1.0 1.0"/>
@@ -125,10 +150,12 @@
       </geometry>
     </collision>
-    <xacro:box_inertia m="10" w="${cond_len}" h="${cond_height}" d="${cond_width}"/>
+    <!-- No origin shift needed here, the parent joint handles it -->
+    <xacro:box_inertia m="10" w="${cond_len}" h="${cond_height}" d="${cond_width}" x="0" y="0" z="0"/>
   </link>
   <joint name="conditioner_joint" type="prismatic">
     <parent link="base_link"/>
     <child link="conditioner_link"/>
-    <origin xyz="${-chassis_len/2 - 0.05} 0 ${-(chassis_height/2) + 0.1}" rpy="0 0 0"/>
+    <!-- Appended + 1.25 to the mathematical Z calculation -->
+    <origin xyz="${-chassis_len/2 - 0.05} 0 ${-(chassis_height/2) + 0.1 + 1.25}" rpy="0 0 0"/>
     <axis xyz="0 0 -1"/>
     <limit lower="0.0" upper="0.5" effort="10000" velocity="0.5"/>
@@ -142,5 +169,6 @@
     <child link="horizontal_auger_link"/>
     <origin xyz="0.2 0 -0.1" rpy="0 1.5708 0"/>
-    <axis xyz="0 0 1"/> <dynamics damping="5.0" friction="10.0"/>
+    <axis xyz="0 0 1"/>
+    <dynamics damping="5.0" friction="10.0"/>
   </joint>
   <link name="vertical_auger_link">
@@ -171,5 +199,6 @@
     <parent link="base_link"/>
     <child link="imu_link"/>
-    <origin xyz="1.5 0 0.8" rpy="0 0 0"/>
+    <!-- Original Z (0.8) + 1.25 = 2.05 -->
+    <origin xyz="1.5 0 2.05" rpy="0 0 0"/>
   </joint>
   <link name="laser_link">
@@ -192,5 +221,6 @@
     <parent link="base_link"/>
     <child link="laser_link"/>
-    <origin xyz="${chassis_len/2 + 0.05} 0 ${-(chassis_height/2) + 0.2}" rpy="0 0 0"/>
+    <!-- Appended + 1.25 to the mathematical Z calculation -->
+    <origin xyz="${chassis_len/2 + 0.05} 0 ${-(chassis_height/2) + 0.2 + 1.25}" rpy="0 0 0"/>
   </joint>
   <ros2_control name="GazeboSimSystem" type="system">
@@ -283,4 +313,7 @@
     <mu1>0.2</mu1> <mu2>0.2</mu2>
     <self_collide>false</self_collide>
+  </gazebo>
+  <gazebo reference="water_tank_link">
+    <material>Gazebo/White</material>
   </gazebo>
   <gazebo reference="rear_left_wheel">
@@ -339,9 +372,8 @@
         <scan>
           <horizontal>
-            <!-- 270 degree FOV -->
             <samples>60</samples>
             <resolution>1.0</resolution>
-            <min_angle>-2.35619</min_angle>
-            <max_angle>2.35619</max_angle>
+            <min_angle>-1</min_angle>
+            <max_angle>1</max_angle>
           </horizontal>
         </scan>
@@ -353,11 +385,11 @@
       </ray>
     </sensor>
-</gazebo>
+  </gazebo>
   <gazebo>
+    <!-- Plugin remains locked strictly to base_link -->
     <plugin filename="gz-sim-odometry-publisher-system" name="gz::sim::systems::OdometryPublisher">
       <odom_frame>odom</odom_frame>
       <robot_base_frame>base_link</robot_base_frame>
       <odom_publish_frequency>50</odom_publish_frequency>
-      <!-- <publish_tf>false</publish_tf>  -->
     </plugin>
   </gazebo>

Commit message: Adjusted lidar and imu positioning

File: ice_resurfacer_description/urdf/ice_resurfacer4.urdf.xacro (robot description, xacro)
@@ -37,5 +37,5 @@
       <origin xyz="-0.5 0.0 0.0" rpy="0 0 0"/>
       <geometry>
-        <mesh filename="package://ice_resurfacer_description/meshes/perfect_body.stl" scale="1 1 1"/>
+        <mesh filename="package://ice_resurfacer_description/meshes/bodywithbumber.stl" scale="1 1 1"/>
       </geometry>
       <material name="blue">
@@ -200,5 +200,5 @@
     <child link="imu_link"/>
     <!-- Original Z (0.8) + 1.25 = 2.05 -->
-    <origin xyz="1.5 0 2.05" rpy="0 0 0"/>
+    <origin xyz="0 0 0.5" rpy="0 0 0"/>
   </joint>
   <link name="laser_link">
@@ -222,5 +222,5 @@
     <child link="laser_link"/>
     <!-- Appended + 1.25 to the mathematical Z calculation -->
-    <origin xyz="${chassis_len/2 + 0.05} 0 ${-(chassis_height/2) + 0.2 + 1.25}" rpy="0 0 0"/>
+    <origin xyz="1.62 0 ${-(chassis_height/2) + 0.2 + 1.25}" rpy="0 0 0"/>
   </joint>
   <ros2_control name="GazeboSimSystem" type="system">
@@ -365,5 +365,5 @@
       <always_on>true</always_on>
       <visualize>true</visualize>
-      <update_rate>1</update_rate>
+      <update_rate>10</update_rate>
       <topic>scan</topic>
       <gz_frame_id>laser_link</gz_frame_id>
@@ -372,13 +372,13 @@
         <scan>
           <horizontal>
-            <samples>60</samples>
+            <samples>90</samples>
             <resolution>1.0</resolution>
-            <min_angle>-1</min_angle>
-            <max_angle>1</max_angle>
+            <min_angle>-1.57079633</min_angle>
+            <max_angle>1.57079633</max_angle>
           </horizontal>
         </scan>
         <range>
           <min>0.4</min>
-          <max>40.0</max>
+          <max>60.0</max>
           <resolution>0.01</resolution>
         </range>

Commit message: further odometry testing, shifting base link to rear axle

File: ice_resurfacer_description/urdf/ice_resurfacer4.urdf.xacro (robot description, xacro)
@@ -35,5 +35,5 @@
   <link name="base_link">
     <visual>
-      <origin xyz="-0.5 0.0 0.0" rpy="0 0 0"/>
+      <origin xyz="0.48 0.0 0.0" rpy="0 0 0"/>
       <geometry>
         <mesh filename="package://ice_resurfacer_description/meshes/bodywithbumber.stl" scale="1 1 1"/>
@@ -44,15 +44,15 @@
     </visual>
     <collision>
-      <origin xyz="0 0 1.55" rpy="0 0 0"/>
+      <origin xyz="0.98 0 1.55" rpy="0 0 0"/>
       <geometry>
         <box size="${chassis_len} ${chassis_width} ${chassis_height - 0.6}"/>
       </geometry>
     </collision>
-    <xacro:box_inertia m="${chassis_mass}" w="${chassis_len}" h="${chassis_height}" d="${chassis_width}" x="0" y="0" z="1.25"/>
+    <xacro:box_inertia m="${chassis_mass}" w="${chassis_len}" h="${chassis_height}" d="${chassis_width}" x="0.98" y="0" z="1.25"/>
   </link>
    <!-- 2. The Water Tank Dummy Link -->
   <link name="water_tank_link">
     <visual>
-      <origin xyz="-0.5 0.0 0.0" rpy="0 0 0"/>
+      <origin xyz="0.48 0.0 0.0" rpy="0 0 0"/>
       <geometry>
         <mesh filename="package://ice_resurfacer_description/meshes/watertank.stl" scale="1 1 1"/>
@@ -89,7 +89,5 @@
       <parent link="base_link"/>
       <child link="${prefix}_wheel"/>
-      <!-- Appended + 1.25 to the mathematical Z calculation -->
-      <origin xyz="${-wheel_base_x} ${reflect * wheel_sep_y} ${wheel_radius - (ground_clearance + chassis_height/2) + 1.25}" rpy="${-pi/2} 0 0"/>
-      <axis xyz="0 0 1"/>
+      <origin xyz="0 ${reflect * wheel_sep_y} ${wheel_radius - (ground_clearance + chassis_height/2) + 1.25}" rpy="${-pi/2} 0 0"/>      <axis xyz="0 0 1"/>
     </joint>
   </xacro:macro>
@@ -106,7 +104,5 @@
       <parent link="base_link"/>
       <child link="${prefix}_steering_link"/>
-      <!-- Appended + 1.25 to the mathematical Z calculation -->
-      <origin xyz="${wheel_base_x} ${reflect * wheel_sep_y} ${wheel_radius - (ground_clearance + chassis_height/2) + 1.25}" rpy="0 0 0"/>
-      <axis xyz="0 0 1"/>
+      <origin xyz="${wheel_base_x * 2} ${reflect * wheel_sep_y} ${wheel_radius - (ground_clearance + chassis_height/2) + 1.25}" rpy="0 0 0"/>      <axis xyz="0 0 1"/>
       <limit lower="-0.6" upper="0.6" effort="50000" velocity="1.0"/>
     </joint>
@@ -156,7 +152,5 @@
     <parent link="base_link"/>
     <child link="conditioner_link"/>
-    <!-- Appended + 1.25 to the mathematical Z calculation -->
-    <origin xyz="${-chassis_len/2 - 0.05} 0 ${-(chassis_height/2) + 0.1 + 1.25}" rpy="0 0 0"/>
-    <axis xyz="0 0 -1"/>
+    <origin xyz="${-chassis_len/2 - 0.05 + 0.98} 0 ${-(chassis_height/2) + 0.1 + 1.25}" rpy="0 0 0"/>    <axis xyz="0 0 -1"/>
     <limit lower="0.0" upper="0.5" effort="10000" velocity="0.5"/>
     <dynamics damping="50.0" friction="50.0"/>
@@ -199,6 +193,5 @@
     <parent link="base_link"/>
     <child link="imu_link"/>
-    <!-- Original Z (0.8) + 1.25 = 2.05 -->
-    <origin xyz="0 0 0.5" rpy="0 0 0"/>
+    <origin xyz="0.98 0 0.5" rpy="0 0 0"/>
   </joint>
   <link name="laser_link">
@@ -222,5 +215,5 @@
     <child link="laser_link"/>
     <!-- Appended + 1.25 to the mathematical Z calculation -->
-    <origin xyz="1.62 0 ${-(chassis_height/2) + 0.2 + 1.25}" rpy="0 0 0"/>
+    <origin xyz="2.60 0 ${-(chassis_height/2) + 0.2 + 1.25}" rpy="0 0 0"/>
   </joint>
   <ros2_control name="GazeboSimSystem" type="system">
@@ -319,28 +312,28 @@
   <gazebo reference="rear_left_wheel">
     <material>Gazebo/DarkGrey</material>
-    <mu1>0.7</mu1> <mu2>0.7</mu2>
+    <mu1>1.0</mu1> <mu2>1.0</mu2>
     <fdir1>1 0 0</fdir1>
-    <kp>100000.0</kp> <kd>500.0</kd>
+    <kp>1000000.0</kp> <kd>500.0</kd>
     <minDepth>0.01</minDepth> <maxVel>0.1</maxVel>
   </gazebo>
   <gazebo reference="rear_right_wheel">
     <material>Gazebo/DarkGrey</material>
-    <mu1>0.7</mu1> <mu2>0.7</mu2>
+    <mu1>1.0</mu1> <mu2>1.0</mu2>
     <fdir1>1 0 0</fdir1>
-    <kp>100000.0</kp> <kd>500.0</kd>
+    <kp>1000000.0</kp> <kd>500.0</kd>
     <minDepth>0.01</minDepth> <maxVel>0.1</maxVel>
   </gazebo>
   <gazebo reference="front_left_wheel">
     <material>Gazebo/DarkGrey</material>
-    <mu1>0.7</mu1> <mu2>0.7</mu2>
+    <mu1>1.0</mu1> <mu2>1.0</mu2>
     <fdir1>1 0 0</fdir1>
-    <kp>100000.0</kp> <kd>500.0</kd>
+    <kp>1000000.0</kp> <kd>500.0</kd>
     <minDepth>0.01</minDepth> <maxVel>0.1</maxVel>
   </gazebo>
   <gazebo reference="front_right_wheel">
     <material>Gazebo/DarkGrey</material>
-    <mu1>0.7</mu1> <mu2>0.7</mu2>
+    <mu1>1.0</mu1> <mu2>1.0</mu2>
     <fdir1>1 0 0</fdir1>
-    <kp>100000.0</kp> <kd>500.0</kd>
+    <kp>1000000.0</kp> <kd>500.0</kd>
     <minDepth>0.01</minDepth> <maxVel>0.1</maxVel>
   </gazebo>
@@ -359,4 +352,5 @@
       <visualize>true</visualize>
       <topic>imu</topic>
+      <gz_frame_id>imu_link</gz_frame_id>
     </sensor>
   </gazebo>

Commit message: Fixed issue with front steering joint. left <--> right

File: ice_resurfacer_description/urdf/ice_resurfacer4.urdf.xacro (robot description, xacro)
@@ -7,5 +7,5 @@
   <xacro:property name="wheel_radius" value="0.386"/>
   <xacro:property name="wheel_width" value="0.215"/>
-  <xacro:property name="wheel_mass" value="50.0"/>
+  <xacro:property name="wheel_mass" value="20.0"/>
   <xacro:property name="wheel_base_x" value="0.98"/>
   <xacro:property name="wheel_sep_y" value="0.685"/>
@@ -14,5 +14,4 @@
   <xacro:property name="cond_height" value="0.3"/>
   <xacro:property name="ground_clearance" value="0.25"/>
-  <!-- UPGRADED MACRO: Now accepts x, y, z to shift the center of mass independently -->
   <xacro:macro name="box_inertia" params="m w h d x y z">
     <inertial>

Commit message: Fixed frame mismatch of the static planner, updated URDF base collision, temporary ground truth

File: ice_resurfacer_description/urdf/ice_resurfacer4.urdf.xacro (robot description, xacro)
@@ -43,7 +43,7 @@
     </visual>
     <collision>
-      <origin xyz="0.98 0 1.55" rpy="0 0 0"/>
-      <geometry>
-        <box size="${chassis_len} ${chassis_width} ${chassis_height - 0.6}"/>
+      <origin xyz="0.50 0 1.55" rpy="0 0 0"/>
+      <geometry>
+        <box size="${chassis_len} ${chassis_width} ${chassis_height - 0.9}"/>
       </geometry>
     </collision>
